Commit message: urdf + position for new flange

File: ros2Packages/src/ur_description/urdf/ur_macro.xacro (robot description, xacro)
@@ -384,5 +384,6 @@
       <!-- origin xyz="0.0552 0.205 0" rpy="0 ${pi/2.0} 0" / -->
       <!-- x is the height offset of 8.47 + 2 cm, y is the other -->
-      <origin xyz="0.1047 0.1544 0" rpy="0 ${pi/2.0} 0" />
+      <!-- origin xyz="0.1047 0.1544 0" rpy="0 ${pi/2.0} 0" / -->
+      <origin xyz="0.1850 0 0" rpy="0 ${pi/2.0} 0" />
     </joint>
   </xacro:macro>

Commit message: Code before final tests
Updated controller, targets depth both in talker and listener, cost function, logs, errors fixed, etc.

File: ros2Packages/src/ur_description/urdf/ur_macro.xacro (robot description, xacro)
@@ -380,11 +380,32 @@
     <link name="${tf_prefix}cstm_flange" />
     <joint name="${tf_prefix}wrist_3_cstm" type="fixed">
-      <parent link="${tf_prefix}flange" />
+      <parent link="${tf_prefix}tool0" />
       <child link="${tf_prefix}cstm_flange" />
       <!-- origin xyz="0.0552 0.205 0" rpy="0 ${pi/2.0} 0" / -->
       <!-- x is the height offset of 8.47 + 2 cm, y is the other -->
       <!-- origin xyz="0.1047 0.1544 0" rpy="0 ${pi/2.0} 0" / -->
+      <origin xyz="0 0 0.1850" rpy="${0} ${0} ${-pi/2.0}" />
+    </joint>
+<!--
+    <link name="${tf_prefix}temp" />
+    <joint name="${tf_prefix}wrist_3_temp" type="fixed">
+      <parent link="${tf_prefix}tool0" />
+      <child link="${tf_prefix}temp" />
+       comment origin xyz="0.0552 0.205 0" rpy="0 ${pi/2.0} 0" /
+       comment x is the height offset of 8.47 + 2 cm, y is the other
+       comment origin xyz="0.1047 0.1544 0" rpy="0 ${pi/2.0} 0" /
+      <origin xyz="0 0 0.1850" rpy="${0} ${0} ${-pi/2.0}" />
+    </joint>
+    Custom Flange
+    <link name="${tf_prefix}cstm_flange" />
+    <joint name="${tf_prefix}wrist_3_cstm" type="fixed">
+      <parent link="${tf_prefix}flange" />
+      <child link="${tf_prefix}cstm_flange" />
+      comment origin xyz="0.0552 0.205 0" rpy="0 ${pi/2.0} 0" /
+      comment x is the height offset of 8.47 + 2 cm, y is the other
+      comment origin xyz="0.1047 0.1544 0" rpy="0 ${pi/2.0} 0" /
       <origin xyz="0.1850 0 0" rpy="0 ${pi/2.0} 0" />
     </joint>
+-->
   </xacro:macro>
 </robot>
